File: hardware/aware01_h7_rev2_0/aware01_h7_rev2_0.kicad_pcb (KiCad board)
At the start: 4 copper layers, 46 x 110 mm, 160 parts, among them IC1 TLV320AIC3204IRHBR, IC2 587-2054-127F, IC3 587-2054-127F, IC4 587-2054-127F, IC5 587-2054-127F, J1 CV3_IN, J10 CV2_IN, J11 V/OCT_IN, J12 CV1_IN, J13 GATE3_IN, J14 GATE4_IN, J2 Conn_02x07_Odd_Even, J3 Conn_02x05_Odd_Even, J4 InL, J5 InR, J6 OutL, J7 OutR, J8 GATE1_IN, J9 GATE2_IN, Q1 MMBT3904, Q2 MMBT3904, Q3 MMBT3904, Q4 MMBT3904, SW1 SW_Push, SW2 SW_Push, SW3 SW_Push, U1 LMR50410Y5FQDBVRQ1, U10 NE5532DRG4, U11 LMV722IDR, U12 LMV722IDR, U2 STM32H7A3RITx, U3 10k, U4 10k, U5 10k, U6 10k, U7 LM1117MP-3.3, U8 LM4040DIM3X-10, U9 NE5532DRG4, Y2 WE-XTAL 24.0MHz 50ppm

Commit message: hw: update hw design
Parts:
- removed C4: 100n, Capacitor_SMD:C_0603_1608Metric
- removed SW1: SW_Push, Eurorack:TS046643BK100SMT
- removed TP10, TP13: TestPoint, TestPoint:TestPoint_Pad_D1.0mm
- added C31: 100n, Capacitor_SMD:C_0603_1608Metric, B.Cu at (153.3, 49.6)
- added C32: 100n, Capacitor_SMD:C_0603_1608Metric, B.Cu at (171.8, 50.8)
- added C34: 100n, Capacitor_SMD:C_0603_1608Metric, B.Cu at (149.4, 50.7)
- added C35: 100n, Capacitor_SMD:C_0603_1608Metric, B.Cu at (138.1, 50.8)
- added R1: 10k, Resistor_SMD:R_0603_1608Metric_Pad0.98x0.95mm_HandSolder, B.Cu at (138.4, 72.0)
- moved C19 0.42 mm to (137.6, 90.0)
- moved Y2 0.35 mm to (134.4, 87.2)
- moved C13 0.11 mm to (134.3, 83.6)
Connections:
- J13 pad TN: unconnected-(J13-PadTN) -> GND
- J14 pad TN: unconnected-(J14-PadTN) -> GND
- J4 pad TN: unconnected-(J4-PadTN) -> GND
- J8 pad TN: unconnected-(J8-PadTN) -> GND
- J9 pad TN: unconnected-(J9-PadTN) -> GND
Routing:
- net /NRST: track 42.0 -> 31.9 mm
- net +5V: track 17.4 -> 20.5 mm, vias 10 -> 18
- net -12V: track 122.5 -> 120.3 mm
- net +3.3VA: track 45.0 -> 46.8 mm
- net GND: track 143.8 -> 145.4 mm
- net +3.3V: track 43.8 -> 45.2 mm, vias 34 -> 40
