File: hardware/aware01_h7_rev2_0/cv_gate.kicad_sch (KiCad schematic)
At the start: 42 parts, among them J10 GATE4_IN, J11 CV2_IN, J12 CV3_IN, J13 V/OCT_IN, J14 CV1_IN, J7 GATE1_IN, J8 GATE2_IN, J9 GATE3_IN, Q1 MMBT3904, Q2 MMBT3904, Q3 MMBT3904, Q4 MMBT3904, U12 OPA2322AIDR, U13 OPA2322AIDR

Commit message: hw: update schematic
Other:
- note added: "Control Interface"
- company: Ausschussware -> Aware Modular
